File: project/project.kicad_pcb (KiCad board)
At the start: 2 copper layers, 100 x 100 mm, 88 parts, among them J1 AC, J2 FAN, J3 transformer, Q1 13001, Q2 S8050, Q3 S8550, Q4 IRF740, Q5 IRF740, SW1 50C NC, SW2 85C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

Commit message: finishing pcb
Parts:
- removed PS1: PSU 12V 1A, Converter_ACDC:Converter_ACDC_HiLink_HLK-PMxx
- removed kibuzzard-64DA8E83: G***, kibuzzard-64DA8E83
- added J2: 12V, TerminalBlock_Phoenix:TerminalBlock_Phoenix_MKDS-1,5-2-5.08_1x02_P5.08mm_Horizontal, F.Cu at (82.7, 116.0)
- added kibuzzard-64DC9B3C: G***, kibuzzard-64DC9B3C, F.Cu at (81.0, 111.0)
- added kibuzzard-64DC9B5D: G***, kibuzzard-64DC9B5D, F.Cu at (170.0, 127.0)
- added kibuzzard-64DC9BC4: G***, kibuzzard-64DC9BC4, F.Cu at (166.0, 67.0)
- added kibuzzard-64DC9C08: G***, kibuzzard-64DC9C08, F.Cu at (80.0, 84.0)
- added kibuzzard-64DCA2D6: G***, kibuzzard-64DCA2D6, F.Cu at (146.5, 138.5)
- added kibuzzard-64DCA30C: G***, kibuzzard-64DCA30C, F.Cu at (80.5, 141.0)
- C21: footprint Capacitor_THT:CP_Radial_D8.0mm_P3.50mm -> Capacitor_SMD:CP_Elec_10x10
- moved G1 151.4 mm to (91.0, 87.0)
- moved R1 136.2 mm to (167.0, 103.2), turned to 90 degrees
- moved RV2 128.0 mm to (94.5, 149.0)
- moved R20 123.4 mm to (93.1, 142.4), turned to 90 degrees
- moved R4 121.8 mm to (169.0, 94.2), turned to -90 degrees
- moved R2 110.6 mm to (169.0, 100.0), turned to -90 degrees
- moved R3 108.4 mm to (167.0, 97.2)
- moved R23 106.9 mm to (118.0, 138.9), turned to -90 degrees
- moved U1 105.9 mm to (81.5, 136.2), turned to 90 degrees
- moved C24 104.0 mm to (116.0, 138.8), turned to 90 degrees
- moved R9 102.6 mm to (91.1, 142.4), turned to -90 degrees
- moved C19 100.7 mm to (95.3, 142.4), turned to 90 degrees
- moved R10 99.9 mm to (89.1, 142.4), turned to 90 degrees
- moved R13 99.3 mm to (93.1, 126.9), turned to -90 degrees
- moved C17 97.3 mm to (87.1, 142.4), turned to -90 degrees
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- renumbered J2 to J3, J3 to J4
Routing:
- net Earth: track 62.2 -> 0.00 mm
- net /ac-dc/12V: track 0.00 -> 59.9 mm
- net /dc-dc/CS: track 0.00 -> 53.1 mm
- net /dc-dc/OUT_L: track 0.00 -> 51.0 mm
- net /dc-dc/COMP: track 0.00 -> 49.4 mm
- net /ac-dc/320V: track 49.9 -> 95.7 mm, vias 0 -> 15
- net +5V: track 0.00 -> 33.7 mm
- net /dc-dc/TX_H: track 43.5 -> 75.9 mm
- net /dc-dc/OUT_H: track 6.93 -> 33.1 mm
- net Net-(C22-Pad1): track 0.00 -> 16.2 mm
- net /dc-dc/HSB: track 15.1 -> 27.2 mm
- net /dc-dc/FB: track 0.00 -> 11.5 mm
- net /dc-dc/HSVcc: track 7.49 -> 18.8 mm, vias 0 -> 2
- net /dc-dc/FAN_12V: track 0.00 -> 9.15 mm
- net Net-(R20-Pad1): track 0.00 -> 8.60 mm
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Other:
- board text added: "+ -"
- board text added: "Current Limit"
- board text added: "D=3mm"
- board text added: "D=4mm"
- board text added: "L GND N"
- board text added: "TXH GND TXL"

Commit message: small power traces rearrangement
Parts:
- moved D7 4.74 mm to (157.5, 123.3)
Routing:
- net /dc-dc/TX_L: track 81.2 -> 65.5 mm
- net GND: track 65.5 -> 56.0 mm
- net /dc-dc/TX_H: track 75.9 -> 79.4 mm
Changed lines of the file:
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@@
   )
   (footprint "Diode_THT:D_DO-201AD_P15.24mm_Horizontal" (layer "F.Cu")
-    (at 157.54 128 -90)
+    (at 157.5 123.26 -90)
     (descr "Diode, DO-201AD series, Axial, Horizontal, pin pitch=15.24mm, , length*diameter=9.5*5.2mm^2, , http://www.diodes.com/_files/packages/DO-201AD.pdf")
     (tags "Diode DO-201AD series Axial Horizontal pin pitch 15.24mm  length 9.5mm diameter 5.2mm")
@@
   (segment (start 94.91 140.9725) (end 95.29 141.3525) (width 0.5) (layer "F.Cu") (net 2))
   (segment (start 153 89.108629) (end 154.38 89.108629) (width 2.5) (layer "F.Cu") (net 2))
-  (segment (start 160.08 132) (end 160.08 140.7) (width 1.5) (layer "F.Cu") (net 2))
+  (segment (start 160.08 135.92) (end 160.08 132) (width 2) (layer "F.Cu") (net 2))
   (segment (start 156.512754 89.487246) (end 156.891371 89.108629) (width 2.5) (layer "F.Cu") (net 2))
-  (segment (start 155 132) (end 155 140.7) (width 1.5) (layer "F.Cu") (net 2))
+  (segment (start 155 136) (end 155 132) (width 2) (layer "F.Cu") (net 2))
+  (segment (start 157.5 138.5) (end 155 136) (width 2) (layer "F.Cu") (net 2))
   (segment (start 154.3925 84.488629) (end 154.3925 89.096129) (width 2.5) (layer "F.Cu") (net 2))
   (segment (start 156.891371 89.108629) (end 159 89.108629) (width 2.5) (layer "F.Cu") (net 2))
@@
   (segment (start 154.38 89.108629) (end 156.891371 89.108629) (width 2.5) (layer "F.Cu") (net 2))
   (segment (start 94.91 138.71) (end 94.91 140.9725) (width 0.5) (layer "F.Cu") (net 2))
+  (segment (start 157.5 138.5) (end 160.08 135.92) (width 2) (layer "F.Cu") (net 2))
   (segment (start 169 93.15) (end 166.85 93.15) (width 0.5) (layer "F.Cu") (net 2))
-  (segment (start 155 140.7) (end 157.54 143.24) (width 1.5) (layer "F.Cu") (net 2))
-  (segment (start 160.08 140.7) (end 157.54 143.24) (width 1.5) (layer "F.Cu") (net 2))
   (segment (start 121 143.015) (end 127 143.015) (width 1.5) (layer "F.Cu") (net 2))
   (via (at 100 139) (size 0.7) (drill 0.3) (layers "F.Cu" "B.Cu") (net 2))
@@
   (segment (start 81.19625 69) (end 86 69) (width 2.5) (layer "F.Cu") (net 28))
   (segment (start 130.5 122.5) (end 154.5 122.5) (width 0.5) (layer "F.Cu") (net 29))
-  (segment (start 166.32 129.015) (end 157.35 129.015) (width 1.5) (layer "F.Cu") (net 29))
   (segment (start 129.9625 123.0375) (end 130.5 122.5) (width 0.5) (layer "F.Cu") (net 29))
-  (segment (start 154.5 122.5) (end 157.54 125.54) (width 0.5) (layer "F.Cu") (net 29))
+  (segment (start 155.26 123.26) (end 157.5 123.26) (width 0.5) (layer "F.Cu") (net 29))
+  (segment (start 169.305 132) (end 160.565 123.26) (width 2) (layer "F.Cu") (net 29))
   (segment (start 129.9625 123.9625) (end 129.9625 123.0375) (width 0.5) (layer "F.Cu") (net 29))
-  (segment (start 157.54 132) (end 157.54 128) (width 1.5) (layer "F.Cu") (net 29))
+  (segment (start 157.54 132) (end 157.54 123.3) (width 2) (layer "F.Cu") (net 29))
+  (segment (start 154.5 122.5) (end 155.26 123.26) (width 0.5) (layer "F.Cu") (net 29))
   (segment (start 144 133.795) (end 146.19 135.985) (width 1.5) (layer "F.Cu") (net 29))
+  (segment (start 157.54 123.3) (end 157.5 123.26) (width 2) (layer "F.Cu") (net 29))
   (segment (start 127.0625 123.9625) (end 129.9625 123.9625) (width 0.5) (layer "F.Cu") (net 29))
   (segment (start 152.19 133.985) (end 152.19 129.985) (width 1.5) (layer "F.Cu") (net 29))
+  (segment (start 160.565 123.26) (end 157.5 123.26) (width 2) (layer "F.Cu") (net 29))
   (segment (start 152.19 129.985) (end 154.175 128) (width 1.5) (layer "F.Cu") (net 29))
-  (segment (start 169.305 132) (end 166.32 129.015) (width 1.5) (layer "F.Cu") (net 29))
   (segment (start 126.025 122.925) (end 127.0625 123.9625) (width 0.5) (layer "F.Cu") (net 29))
   (segment (start 154.175 128) (end 157.54 128) (width 1.5) (layer "F.Cu") (net 29))
-  (segment (start 157.54 125.54) (end 157.54 128) (width 0.5) (layer "F.Cu") (net 29))
   (segment (start 150.19 135.985) (end 152.19 133.985) (width 1.5) (layer "F.Cu") (net 29))
   (segment (start 146.19 135.985) (end 150.19 135.985) (width 1.5) (layer "F.Cu") (net 29))
   (segment (start 144 132) (end 144 133.795) (width 1.5) (layer "F.Cu") (net 29))
-  (segment (start 138 132.015) (end 138 140.715) (width 1.5) (layer "F.Cu") (net 30))
-  (segment (start 155.065001 152.860001) (end 152.19 149.985) (width 1.5) (layer "F.Cu") (net 30))
-  (segment (start 152.19 149.985) (end 152.19 146.985) (width 1.5) (layer "F.Cu") (net 30))
+  (segment (start 138 140.715) (end 138 135) (width 2.5) (layer "F.Cu") (net 30))
+  (segment (start 166 142.5) (end 148 142.5) (width 2.5) (layer "F.Cu") (net 30))
+  (segment (start 138 135) (end 132.985 135) (width 1.5) (layer "F.Cu") (net 30))
+  (segment (start 148 142.5) (end 140.5 135) (width 2.5) (layer "F.Cu") (net 30))
+  (segment (start 132.985 135) (end 132.92 134.935) (width 1.5) (layer "F.Cu") (net 30))
+  (segment (start 166.5 142) (end 166 142.5) (width 2.5) (layer "F.Cu") (net 30))
+  (segment (start 124.46 132.015) (end 124.46 133.475) (width 1.5) (layer "F.Cu") (net 30))
+  (segment (start 169.305 142) (end 166.5 142) (width 2.5) (layer "F.Cu") (net 30))
+  (segment (start 138 132.015) (end 138 135) (width 1.5) (layer "F.Cu") (net 30))
+  (segment (start 135.46 143.255) (end 138 140.715) (width 2.5) (layer "F.Cu") (net 30))
+  (segment (start 140.5 135) (end 138 135) (width 2.5) (layer "F.Cu") (net 30))
+  (segment (start 125.92 134.935) (end 132.92 134.935) (width 1.5) (layer "F.Cu") (net 30))
   (segment (start 132.92 132.015) (end 132.92 134.935) (width 1.5) (layer "F.Cu") (net 30))
-  (segment (start 124.46 132.015) (end 124.46 133.475) (width 1.5) (layer "F.Cu") (net 30))
-  (segment (start 132.92 134.935) (end 132.92 140.715) (width 1.5) (layer "F.Cu") (net 30))
-  (segment (start 138 140.715) (end 135.46 143.255) (width 1.5) (layer "F.Cu") (net 30))
-  (segment (start 152.19 146.985) (end 145.92 140.715) (width 1.5) (layer "F.Cu") (net 30))
-  (segment (start 160.314999 152.860001) (end 155.065001 152.860001) (width 1.5) (layer "F.Cu") (net 30))
-  (segment (start 165.175 142) (end 169.305 142) (width 1.5) (layer "F.Cu") (net 30))
-  (segment (start 145.92 140.715) (end 138 140.715) (width 1.5) (layer "F.Cu") (net 30))
-  (segment (start 163.19 143.985) (end 165.175 142) (width 1.5) (layer "F.Cu") (net 30))
-  (segment (start 132.92 140.715) (end 135.46 143.255) (width 1.5) (layer "F.Cu") (net 30))
-  (segment (start 125.92 134.935) (end 132.92 134.935) (width 1.5) (layer "F.Cu") (net 30))
-  (segment (start 163.19 149.985) (end 160.314999 152.860001) (width 1.5) (layer "F.Cu") (net 30))
-  (segment (start 163.19 143.985) (end 163.19 149.985) (width 1.5) (layer "F.Cu") (net 30))
   (segment (start 124.46 133.475) (end 125.92 134.935) (width 1.5) (layer "F.Cu") (net 30))
   (segment (start 128.485 132.015) (end 130 130.5) (width 0.5) (layer "F.Cu") (net 31))
@@
   (group "" (id 963164d0-a38f-46e1-99b7-939be5f3c834)
     (members
+      131b549b-3dc1-46c8-bd92-e56ac791c494
       15d246eb-24b1-40a1-833b-3d6ec760c1d7
-      19233606-1d28-4fe2-888e-adb7f5e868d2
+      2f08b91b-b82a-4412-845d-b1b59b1b0ea5
+      3e8f0ecf-3485-49de-b30b-ae58d17d5606
       4d2c8421-35a2-4cac-9e83-b2dc98b8f398
-      6871b399-e370-4f5f-a096-2c1e7ff58751
-      b3686b87-95d8-4df6-a107-58ab07aad67b
+      aa5f6021-f505-4563-8411-d276ce16be3d
+      add6761a-ab0d-487c-8bec-31d31f02c196
+      d2c24d8f-6b3e-4124-a3c2-48164d0a589a
       f554aad4-3598-4db5-b80d-76ac516eda81
     )
@@
   (group "" (id bb6cd49e-661f-4a07-ad46-109e5265b355)
     (members
-      5773b11c-2a82-4fb0-a26c-2e199722bba7
-      5b68be82-2600-4d92-a3c0-6749529b22c2
-      6f5cd6f1-541a-44b3-b3a1-865ff11c57b7
+      48eb36b9-ea71-4c88-ad82-873c0f1ee52c
+      4af9bcd8-746b-40ca-9454-9d397f23c601
+      73fa6f95-911a-4c52-b2e6-eb04eba9554a
+      76b19efd-22b0-4841-83da-59be629218ae
+      99e62952-58b5-4340-941e-ef3e0f4e23ec
       a768ca6d-27cd-4251-8f0d-c3b3f9d71583
+      d38ed290-cf6c-4bf3-b3ec-417649164947
       de39f8f9-9558-4db5-a511-0bec5fd411f0
-      ebbe3aa5-6860-49d6-8a39-6d93ecc5c41b
-      f2845290-42a3-47ae-93c4-aa603855aac8
-    )
-  )
+    )
+  )
