File: project/_dc-dc.kicad_sch (KiCad schematic)
At the start: 28 parts

Commit message: adding more things and specifying components
Parts:
- removed D? (x2): UF5408, Diode_THT:D_DO-201AD_P15.24mm_Horizontal, symbol Diode:UF5408
- added C?: 1u, Capacitor_SMD:C_0805_2012Metric_Pad1.18x1.45mm_HandSolder, symbol Device:C
- added C?: 100n, Capacitor_SMD:C_0805_2012Metric_Pad1.18x1.45mm_HandSolder, symbol Device:C
- added D? (x2): MURF1040GCT, Package_TO_SOT_THT:TO-220-3_Horizontal_TabUp, symbol Device:D_Dual_CommonCathode_AKA_Parallel
- added D?: S2M, Diode_SMD:D_SMA_Handsoldering, symbol Diode:UF5408
- added Q?: 13001, Package_TO_SOT_SMD:SOT-23, symbol Device:Q_NPN_BEC
- added Q?: S8050, Package_TO_SOT_SMD:SOT-23, symbol Device:Q_NPN_BEC
- added Q?: S8550, Package_TO_SOT_SMD:SOT-23, symbol Device:Q_PNP_BEC
- added R? (x4): 1k, Resistor_SMD:R_0805_2012Metric_Pad1.20x1.40mm_HandSolder, symbol Device:R
- added R?: 10k, Resistor_SMD:R_0805_2012Metric_Pad1.20x1.40mm_HandSolder, symbol Device:R
- added R?: 10, Resistor_SMD:R_0805_2012Metric_Pad1.20x1.40mm_HandSolder, symbol Device:R
- C?: value 10u/16v -> 10u; Value2 (none) -> 10v
- C?: value 100u/35v -> 100u; Value2 (none) -> 16v
- Q? (x2): footprint Package_TO_SOT_THT:TO-220-3_Vertical -> Package_TO_SOT_THT:TO-220-3_Horizontal_TabUp
- R? (x5): value 0.1 -> 0R1
Connections:
- net GND: now also C?.2, D?.1 (K), D?.3 (K)
- net at Q?.2 (D), TR?.13: now also D?.1 (K), D?.3 (K)
- net at Q?.3 (S), TR?.14: now also C?.2, D?.2 (A), Q?.3 (C)
- net at R?.2: now also U?.6 (OUT), R?.2
- net 12V: now reaches C?.1, C?.1, U?.7 (VCC)
- net 12V: now also D?.2 (A), R?.2
- net at R?.2: now also Q?.2 (E), Q?.2 (E)
- net VCC renamed 320V
- net 320V: now also D?.2 (A)
- new net: C?.1, D?.1 (K), Q?.3 (C), R?.1, R?.1
- new net: R?.1, R?.1, R?.2, R?.2
- new net: C?.1, Q?.1 (B), R?.1
- new net: Q?.2 (E), R?.1
- new net: Q?.1 (B), Q?.1 (B), Q?.3 (C), R?.2, R?.2
Other:
- note added: "todo: * fan power with thermo relay * universal transformer footprint"
- moved on the sheet: C?, Q?, R?, RV?, TR?

Commit message: starting pcb
Parts:
- removed TR?: TEZ16.0-D-2, Transformer_THT:Transformer_Breve_TEZ-47x57, symbol Transformer:TEZ16.0-D-2
- added D10, D7: UF5408, Diode_THT:D_DO-201AD_P15.24mm_Horizontal, symbol Diode:1N5408
- added J2: FAN, Connector_Molex:Molex_KK-254_AE-6410-03A_1x03_P2.54mm_Vertical, symbol Connector_Generic:Conn_01x03
- added J3: transformer, TerminalBlock_Phoenix:TerminalBlock_Phoenix_MKDS-1,5-3_1x03_P5.00mm_Horizontal, symbol Connector:Screw_Terminal_01x03
- added SW1: 50C NC, -local:TO-220-2_Horizontal_TabUp, symbol Switch:SW_SPST_Temperature
- added SW2: 85C, -local:TO-220-2_Horizontal_TabUp, symbol Switch:SW_SPST_Temperature
- D8, D9: renamed from D?; footprint Package_TO_SOT_THT:TO-220-3_Horizontal_TabUp -> -local:TO-220-3_Horizontal_TabUp
- Q4, Q5: renamed from Q?; footprint Package_TO_SOT_THT:TO-220-3_Horizontal_TabUp -> -local:TO-220-3_Horizontal_TabUp
- RV2: renamed from RV?; footprint (none) -> Potentiometer_THT:Potentiometer_Bourns_3296W_Vertical
- U1: renamed from U?; LCSC# (none) -> C109226
- gave numbers to parts that had none: 33
Connections:
- net 12V: now also SW1.1 (A)
- net 320V: now also D10.1 (K)
- net GND: now also D7.2 (A), J2.1 (Pin_1), SW2.1 (A)
- net TX_H: now reaches C23.2, D8.2 (A), Q3.3 (C), Q4.3 (S)
- net TX_H: now also D7.1 (K), J3.3 (Pin_3)
- net HSVcc: now reaches C23.1, D6.1 (K), Q2.3 (C), R15.1, R17.1
- net Gate_L: now reaches Q5.1 (G), R22.1
- net TX_L: now reaches D9.1 (K), D9.3 (K), Q5.2 (D)
- net TX_L: now also D10.2 (A), J3.1 (Pin_1)
- net SHUNT: now reaches Q5.3 (S), R23.1, R24.1, R25.1, R26.1, R27.1, R28.1
- net FB: now reaches C18.2, R12.1, U2.2 (FB)
- net OUT_L: now reaches R19.2, R22.2, U2.6 (OUT)
- net COMP: now reaches R13.2, U2.1 (COMP)
- net COMP: now also SW2.2 (B)
- net CS: now reaches C24.1, R23.2, RV2.1, U2.3 (CS)
- net RC: now reaches C17.1, R10.2, U2.4 (RC)
- net HSB: now reaches Q1.3 (C), Q2.1 (B), Q3.1 (B), R16.2, R18.2
- net Gate_H: now reaches Q4.1 (G), R21.1
- net OUT_H: now reaches Q2.2 (E), Q3.2 (E), R21.2
- new net Earth: J3.2 (Pin_2)
- new net FAN_12V: J2.2 (Pin_2), SW1.2 (B)
- no-connect marks 0 -> 3
Other:
- note added: "Gate Drivers"
- note added: "Power Stage"
- note added: "Primary Current Feedback shunt 20mR 0.3W 80mV@4A"
- note added: "Secondary Voltage Feedback"
- note added: "Switching frequency Fosc=1.72/(R*C) 1.72/((15k+2k2)*1n)=100khz Fsw=50khz"
- note added: "Thermal Fan Control"
- note added: "Thermal Shutdown"
- note removed: "80mV@4A 20mR 0.3W"
- note removed: "Fosc=1.72/(R*C) 1.72/((15k+2k2)*1n)=100khz Fsw=50khz"
- note removed: "todo: * fan power with thermo relay * universal transformer footprint"
- company: (none) -> makerspace.lt
- title: (none) -> psu-500-pri
- moved on the sheet: C17, C18, C19, C22, C23, D6, D8, D9, Q1, Q2, Q3, Q4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

Commit message: finishing pcb
Parts:
- C21: footprint Capacitor_THT:CP_Radial_D8.0mm_P3.50mm -> Capacitor_SMD:CP_Elec_10x10
- renumbered J2 to J3, J3 to J4
Changed lines of the file:
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@@
   (symbol (lib_id "-local:+5V") (at 88.9 132.08 0) (unit 1)
     (in_bom yes) (on_board yes)
-    (property "Reference" "#PWR018" (id 0) (at 88.9 135.89 0)
+    (property "Reference" "#PWR017" (id 0) (at 88.9 135.89 0)
       (effects (font (size 1.27 1.27)) hide)
     )
@@
   (symbol (lib_id "-local:GND") (at 50.8 135.89 0) (unit 1)
     (in_bom yes) (on_board yes) (fields_autoplaced)
-    (property "Reference" "#PWR015" (id 0) (at 50.8 142.24 0)
+    (property "Reference" "#PWR014" (id 0) (at 50.8 142.24 0)
       (effects (font (size 1.27 1.27)) hide)
     )
@@
   (symbol (lib_id "-local:GND") (at 60.96 45.72 0) (unit 1)
     (in_bom yes) (on_board yes) (fields_autoplaced)
-    (property "Reference" "#PWR017" (id 0) (at 60.96 52.07 0)
+    (property "Reference" "#PWR016" (id 0) (at 60.96 52.07 0)
       (effects (font (size 1.27 1.27)) hide)
     )
@@
   (symbol (lib_id "-local:GND") (at 38.1 78.74 0) (unit 1)
     (in_bom yes) (on_board yes) (fields_autoplaced)
-    (property "Reference" "#PWR013" (id 0) (at 38.1 85.09 0)
+    (property "Reference" "#PWR012" (id 0) (at 38.1 85.09 0)
       (effects (font (size 1.27 1.27)) hide)
     )
@@
   (symbol (lib_id "-local:GND") (at 54.61 182.88 0) (unit 1)
     (in_bom yes) (on_board yes) (fields_autoplaced)
-    (property "Reference" "#PWR016" (id 0) (at 54.61 189.23 0)
+    (property "Reference" "#PWR015" (id 0) (at 54.61 189.23 0)
       (effects (font (size 1.27 1.27)) hide)
     )
@@
   (symbol (lib_id "-local:+5V") (at 48.26 121.92 0) (unit 1)
     (in_bom yes) (on_board yes)
-    (property "Reference" "#PWR014" (id 0) (at 48.26 125.73 0)
+    (property "Reference" "#PWR013" (id 0) (at 48.26 125.73 0)
       (effects (font (size 1.27 1.27)) hide)
     )
@@
   (symbol (lib_id "Connector_Generic:Conn_01x03") (at 66.04 40.64 0) (mirror x) (unit 1)
     (in_bom yes) (on_board yes) (fields_autoplaced)
-    (property "Reference" "J2" (id 0) (at 66.04 31.75 0))
+    (property "Reference" "J3" (id 0) (at 66.04 31.75 0))
     (property "Value" "FAN" (id 1) (at 66.04 34.29 0))
     (property "Footprint" "Connector_Molex:Molex_KK-254_AE-6410-03A_1x03_P2.54mm_Vertical" (id 2) (at 66.04 40.64 0)
@@
   (symbol (lib_id "-local:GND") (at 128.27 73.66 0) (unit 1)
     (in_bom yes) (on_board yes) (fields_autoplaced)
-    (property "Reference" "#PWR023" (id 0) (at 128.27 80.01 0)
+    (property "Reference" "#PWR022" (id 0) (at 128.27 80.01 0)
       (effects (font (size 1.27 1.27)) hide)
     )
@@
   (symbol (lib_id "-local:Earth") (at 243.84 67.31 0) (unit 1)
     (in_bom yes) (on_board yes) (fields_autoplaced)
-    (property "Reference" "#PWR0101" (id 0) (at 243.84 73.66 0)
+    (property "Reference" "#PWR026" (id 0) (at 243.84 73.66 0)
       (effects (font (size 1.27 1.27)) hide)
     )
@@
   (symbol (lib_id "Connector:Screw_Terminal_01x03") (at 252.73 66.04 0) (mirror x) (unit 1)
     (in_bom yes) (on_board yes)
-    (property "Reference" "J3" (id 0) (at 251.46 59.69 0)
+    (property "Reference" "J4" (id 0) (at 251.46 59.69 0)
       (effects (font (size 1.27 1.27)) (justify left))
     )
@@
       (effects (font (size 1.27 1.27)) (justify left))
     )
-    (property "Footprint" "Capacitor_THT:CP_Radial_D8.0mm_P3.50mm" (id 2) (at 117.8052 119.38 0)
+    (property "Footprint" "Capacitor_SMD:CP_Elec_10x10" (id 2) (at 117.8052 119.38 0)
       (effects (font (size 1.27 1.27)) hide)
     )
@@
   (symbol (lib_id "-local:GND") (at 101.6 140.97 0) (unit 1)
     (in_bom yes) (on_board yes) (fields_autoplaced)
-    (property "Reference" "#PWR019" (id 0) (at 101.6 147.32 0)
+    (property "Reference" "#PWR018" (id 0) (at 101.6 147.32 0)
       (effects (font (size 1.27 1.27)) hide)
     )
@@
   (symbol (lib_id "-local:GND") (at 198.12 146.05 0) (unit 1)
     (in_bom yes) (on_board yes) (fields_autoplaced)
-    (property "Reference" "#PWR025" (id 0) (at 198.12 152.4 0)
+    (property "Reference" "#PWR024" (id 0) (at 198.12 152.4 0)
       (effects (font (size 1.27 1.27)) hide)
     )
@@
   (symbol (lib_id "-local:GND") (at 212.09 129.54 0) (unit 1)
     (in_bom yes) (on_board yes) (fields_autoplaced)
-    (property "Reference" "#PWR026" (id 0) (at 212.09 135.89 0)
+    (property "Reference" "#PWR025" (id 0) (at 212.09 135.89 0)
       (effects (font (size 1.27 1.27)) hide)
     )
@@
   (symbol (lib_id "-local:GND") (at 101.6 161.29 0) (unit 1)
     (in_bom yes) (on_board yes) (fields_autoplaced)
-    (property "Reference" "#PWR021" (id 0) (at 101.6 167.64 0)
+    (property "Reference" "#PWR020" (id 0) (at 101.6 167.64 0)
       (effects (font (size 1.27 1.27)) hide)
     )
@@
   (symbol (lib_id "-local:+5V") (at 181.61 119.38 0) (unit 1)
     (in_bom yes) (on_board yes)
-    (property "Reference" "#PWR024" (id 0) (at 181.61 123.19 0)
+    (property "Reference" "#PWR023" (id 0) (at 181.61 123.19 0)
       (effects (font (size 1.27 1.27)) hide)
     )
@@
   (symbol (lib_id "-local:+5V") (at 29.21 173.99 0) (unit 1)
     (in_bom yes) (on_board yes)
-    (property "Reference" "#PWR012" (id 0) (at 29.21 177.8 0)
+    (property "Reference" "#PWR011" (id 0) (at 29.21 177.8 0)
       (effects (font (size 1.27 1.27)) hide)
     )
@@
   (symbol (lib_id "-local:GND") (at 106.68 119.38 0) (unit 1)
     (in_bom yes) (on_board yes) (fields_autoplaced)
-    (property "Reference" "#PWR022" (id 0) (at 106.68 125.73 0)
+    (property "Reference" "#PWR021" (id 0) (at 106.68 125.73 0)
       (effects (font (size 1.27 1.27)) hide)
     )
@@
   (symbol (lib_id "-local:+5V") (at 101.6 153.67 0) (unit 1)
     (in_bom yes) (on_board yes)
-    (property "Reference" "#PWR020" (id 0) (at 101.6 157.48 0)
-      (effects (font (size 1.27 1.27)) hide)
-    )
+    (property "Reference" "#PWR019" (id 0) (at 101.6 157.48 0)
+      (effects (font (size 1.27 1.27)) hide)
+    )

Commit message: adding few part numbers to the bom
Parts:
- Q4, Q5: LCSC# (none) -> C2980280
- U2: value UC3845_DIP8 -> UC3845B; LCSC# (none) -> C347460
Changed lines of the file:
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@@
+      (effects (font (size 1.27 1.27)) hide)
+    )
+    (property "jlc-part-type" "" (id 5) (at 212.09 68.58 0)
       (effects (font (size 1.27 1.27)) hide)
     )
@@
       (effects (font (size 1.27 1.27) italic) (justify left) hide)
     )
-    (property "Datasheet" "http://www.vishay.com/docs/91054/91054.pdf" (id 3) (at 222.25 81.28 0)
+    (property "Datasheet" "https://datasheet.lcsc.com/lcsc/2203231030_Minos-IRF740_C2980280.pdf" (id 3) (at 222.25 81.28 0)
       (effects (font (size 1.27 1.27)) (justify left) hide)
+    )
+    (property "LCSC#" "C2980280" (id 4) (at 222.25 81.28 0)
+      (effects (font (size 1.27 1.27)) hide)
+    )
+    (property "jlc-part-type" "" (id 5) (at 222.25 81.28 0)
+      (effects (font (size 1.27 1.27)) hide)
     )
     (pin "1")
@@
       (effects (font (size 1.27 1.27)) (justify left))
     )
-    (property "Value" "UC3845_DIP8" (id 1) (at 102.87 140.97 0)
+    (property "Value" "UC3845B" (id 1) (at 102.87 140.97 0)
       (effects (font (size 1.27 1.27)) (justify left))
     )
@@
       (effects (font (size 1.27 1.27)) hide)
     )
-    (property "Datasheet" "http://www.ti.com/lit/ds/symlink/uc3842.pdf" (id 3) (at 101.6 130.81 0)
+    (property "Datasheet" "https://datasheet.lcsc.com/lcsc/2007031829_UMW-Youtai-Semiconductor-Co---Ltd--UC3845B_C347460.pdf" (id 3) (at 101.6 130.81 0)
+      (effects (font (size 1.27 1.27)) hide)
+    )
+    (property "LCSC#" "C347460" (id 4) (at 101.6 130.81 0)
+      (effects (font (size 1.27 1.27)) hide)
+    )
+    (property "jlc-part-type" "" (id 5) (at 101.6 130.81 0)
       (effects (font (size 1.27 1.27)) hide)
     )
@@
     )
     (property "Value2" "400V" (id 5) (at 144.78 67.31 0))
+    (property "jlc-part-type" "" (id 6) (at 137.16 63.5 0)
+      (effects (font (size 1.27 1.27)) hide)
+    )
     (pin "1")
     (pin "2")
@@
       (effects (font (size 1.27 1.27)) hide)
     )
+    (property "jlc-part-type" "" (id 5) (at 36.83 125.73 0)
+      (effects (font (size 1.27 1.27)) hide)
+    )
     (pin "1")
     (pin "2")
@@
       (effects (font (size 1.27 1.27) italic) (justify left) hide)
     )
-    (property "Datasheet" "http://www.vishay.com/docs/91054/91054.pdf" (id 3) (at 209.55 48.26 0)
+    (property "Datasheet" "https://datasheet.lcsc.com/lcsc/2203231030_Minos-IRF740_C2980280.pdf" (id 3) (at 209.55 48.26 0)
       (effects (font (size 1.27 1.27)) (justify left) hide)
+    )
+    (property "LCSC#" "C2980280" (id 4) (at 209.55 48.26 0)
+      (effects (font (size 1.27 1.27)) hide)
+    )
+    (property "jlc-part-type" "" (id 5) (at 209.55 48.26 0)
+      (effects (font (size 1.27 1.27)) hide)
     )
     (pin "1")
@@
       (effects (font (size 1.27 1.27)) hide)
     )
+    (property "jlc-part-type" "" (id 4) (at 198.12 142.24 0)
+      (effects (font (size 1.27 1.27)) hide)
+    )
     (pin "1")
     (pin "2")
@@
       (effects (font (size 1.27 1.27)) hide)
     )
+    (property "jlc-part-type" "" (id 5) (at 224.79 66.04 0)
+      (effects (font (size 1.27 1.27)) hide)
+    )
