File: project/project.kicad_sch (KiCad schematic)
At the start: 6 parts

Commit message: adding more things and specifying components
Other:
- sheet ac-dc ports: added 12V, 320V; removed none
- sheet dc-dc ports: added 12V, 320V; removed none

Commit message: starting pcb
Parts:
- gave numbers to parts that had none: 4
Connections:
- net Earth: now reaches H3.1
- net Earth: now also H1.1, H2.1, H4.1
Other:
- moved on the sheet: H1, H2, H3, H4

Commit message: finalizing pcb and adding gerbers
Parts:
- added SYM1: SYM_Flash_Small, -local:qr, symbol Graphic:SYM_Flash_Small
Changed lines of the file:
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@@
     (pin "1")
+  )
+  (symbol (lib_id "Graphic:SYM_Flash_Small") (at 30.48 186.69 0) (unit 1)
+    (in_bom yes) (on_board yes) (fields_autoplaced)
+    (property "Reference" "SYM1" (id 0) (at 28.194 186.69 90)
+      (effects (font (size 1.27 1.27)) hide)
+    )
+    (property "Value" "SYM_Flash_Small" (id 1) (at 32.766 186.69 90)
+      (effects (font (size 1.27 1.27)) hide)
+    )
+    (property "Footprint" "-local:qr" (id 2) (at 30.48 187.325 0)
+      (effects (font (size 1.27 1.27)) hide)
+    )
+    (property "Datasheet" "~" (id 3) (at 40.64 189.23 0)
+      (effects (font (size 1.27 1.27)) hide)
+    )
   )
   (symbol (lib_id "power:PWR_FLAG") (at 114.3 190.5 0) (unit 1)
@@
       (reference "SW2") (unit 1) (value "85C") (footprint "-local:TO-220-2_Horizontal_TabUp")
     )
+    (path "/1ec9ce39-046d-4a61-a3a4-f68134989604"
+      (reference "SYM1") (unit 1) (value "SYM_Flash_Small") (footprint "-local:qr")
+    )
     (path "/39a95302-f23d-46b1-ac1d-072d6571958e/e0ef855f-c38d-4374-86a8-8b8c4c9443d6"
